Commit message: .

File: src/spiderbot_description/urdf/spidy.urdf (robot description, URDF)
Before this commit: robot spiderbot, 13 links, 12 joints
Joints:
- joint fl_tibia_joint: axis -0.707107 -0.707107 0.0 -> 0.707107 0.707107 0.0

File: src/spiderbot_description/urdf/spidy.xacro (robot description, xacro)
@@ -315,5 +315,5 @@
   <parent link="fl_femur_link"/>
   <child link="fl_tibia_link"/>
-  <axis xyz="-0.707107 -0.707107 0.0"/>
+  <axis xyz="0.707107 0.707107 0.0"/>
   <limit upper="1.570796" lower="-1.570796" effort="100" velocity="10"/>
   <dynamics damping="0.1" friction="0.1"/>
