Commit message: for slam

File: src/spiderbot_description/urdf/old_correct.urdf (robot description, URDF)
Before this commit: robot spiderbot, 14 links, 13 joints
Links:
- removed link laser_link
Joints:
- removed joint laser_joint

File: src/spiderbot_description/urdf/spidy.xacro (robot description, xacro)
@@ -546,3 +546,62 @@
   </sensor>
 </gazebo>
+<!-- ============================================ -->
+<!-- 2D LIDAR SENSOR -->
+<!-- ============================================ -->
+<link name="laser_link">
+  <inertial>
+    <mass value="0.125"/>
+    <origin xyz="0 0 0" rpy="0 0 0"/>
+    <inertia ixx="0.001" iyy="0.001" izz="0.001"
+             ixy="0.0" ixz="0.0" iyz="0.0"/>
+  </inertial>
+  <visual>
+    <origin xyz="0 0 0" rpy="0 0 0"/>
+    <geometry>
+      <cylinder radius="0.03" length="0.04"/>
+    </geometry>
+    <material name="black"/>
+  </visual>
+  <collision>
+    <origin xyz="0 0 0" rpy="0 0 0"/>
+    <geometry>
+      <cylinder radius="0.03" length="0.04"/>
+    </geometry>
+  </collision>
+</link>
+<!-- Mount LIDAR on top of base_link -->
+<joint name="laser_joint" type="fixed">
+  <origin xyz="0.0 0.0 0.05" rpy="0 0 0"/>
+  <parent link="base_link"/>
+  <child link="laser_link"/>
+</joint>
+<!-- Gazebo LIDAR Plugin -->
+<gazebo reference="laser_link">
+  <sensor name="lidar_sensor" type="gpu_lidar">
+    <topic>scan</topic>
+    <update_rate>10</update_rate>
+    <lidar>
+      <scan>
+        <horizontal>
+          <samples>360</samples>
+          <resolution>1.0</resolution>
+          <min_angle>-3.14159</min_angle>
+          <max_angle>3.14159</max_angle>
+        </horizontal>
+      </scan>
+      <range>
+        <min>0.12</min>
+        <max>12.0</max>
+        <resolution>0.01</resolution>
+      </range>
+      <noise>
+        <type>gaussian</type>
+        <mean>0.0</mean>
+        <stddev>0.01</stddev>
+      </noise>
+    </lidar>
+    <always_on>true</always_on>
+    <visualize>true</visualize>
+  </sensor>
+</gazebo>
 </robot>
